File: Tympan_D.kicad_pcb (KiCad board)
At the start: 4 copper layers, 38 x 74 mm, 116 parts, among them IC1 MK66FX1M0VMD18, IC2 MKL02Z32VFG4, IC3 BC127, J1 SJ-3523-SMT-TR, J2 SJ-3524-SMT-TR-PI, J3 alt Power Pads, P1 USB_OTG, P10 CONN_01X01, P2 CONN_01X06, P3 CONN_01X06, P4 CONN_01X06, P5 CONN_01X06, P6 CONN_01X03, P7 CONN_01X01, P8 CONN_01X01, P9 CONN_01X01, SW1 CL-SB-22A, SW2 TACT_SWITCH, U1 AP2210K-3.3TRG1, U2 TLV320AIC3206IRSBT, U3 74LVC1G66, U4 LP5907MFX-1.8, U5 MCP73831, Y1 32.768kHz, Y2 16MHz

Commit message: tightened solder mask around pads per CM recommendation
Other:
- rule pad_to_mask_clearance: 0.2 -> 0.05
- rule solder_mask_min_width: 0.25 -> 0.02
Changed lines of the file:
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@@
   (layers
     (0 F.Cu signal)
-    (1 In1.Cu power)
-    (2 In2.Cu mixed)
+    (1 In1.Cu power hide)
+    (2 In2.Cu mixed hide)
     (31 B.Cu signal)
     (32 B.Adhes user)
@@
     (pad_size 1.5 3.4)
     (pad_drill 0)
-    (pad_to_mask_clearance 0.2)
-    (solder_mask_min_width 0.25)
+    (pad_to_mask_clearance 0.05)
+    (solder_mask_min_width 0.02)
     (aux_axis_origin 114.85 120.48)
     (grid_origin 114.85 120.48)
     (visible_elements FFFDFFFF)
     (pcbplotparams
-      (layerselection 0x010fc_ffffffff)
+      (layerselection 0x000c0_7ffffff8)
       (usegerberextensions false)
       (usegerberattributes false)
